Commit message: urdf + observation 72

File: resources/robots/go1_widowx/urdf/go1_widowx.urdf (robot description, URDF)
Before this commit: robot go1_widowx, 37 links, 36 joints
Joints:
- removed joint forearm_roll
- added joint widow_forearm_roll: type revolute, parent wx250s/upper_forearm_link, child wx250s/lower_forearm_link, origin xyz=0.175 0 0 rpy=0 0 0, axis 1 0 0, limit lower=-3.141582653589793 upper=3.141582653589793 effort=2 velocity=3.141592653589793
- joint gripper: type continuous -> fixed
- joint widow_left_finger: type prismatic -> fixed
- joint widow_right_finger: type prismatic -> fixed
